Commit message: Fixed disjoint camera link

File: gym_dofbot/envs/arm.urdf (robot description, URDF)
Before this commit: robot arm, 6 links, 5 joints
Links:
- removed link link4
- removed link link5
- added link camera_base, mass 0.00001; collision mesh filename=meshes/link4.STL; visual mesh filename=meshes/link4.STL
- added link camera_lens; collision mesh filename=meshes/camera_lens.STL; visual mesh filename=meshes/camera_lens.STL
- added link camera_target; visual mesh filename=meshes/camera_lens.STL
- added link grasp_target; visual mesh filename=meshes/camera_lens.STL
- added link gripper; collision mesh filename=meshes/link5.STL; visual mesh filename=meshes/link5.STL
Joints:
- added joint joint6: type fixed, parent camera_base, child camera_lens, origin xyz=-0.05385 -0.0645 -0.0075 rpy=0 -1.57 0, axis 0 0 1, limit lower=-1.5708 upper=3.1416 effort=30 velocity=1.0
- added joint joint7: type fixed, parent camera_lens, child camera_target, origin xyz=0 0 0.1 rpy=0 0 0, axis 0 0 1, limit lower=-1.5708 upper=3.1416 effort=30 velocity=1.0
- added joint joint8: type fixed, parent camera_lens, child grasp_target, origin xyz=0 0.06 0.1 rpy=0 0 0, axis 0 0 1, limit lower=-1.5708 upper=3.1416 effort=30 velocity=1.0
- joint joint4: child link4 -> camera_base
- joint joint5: child link5 -> gripper; parent link4 -> camera_base
